File: PCB/CT_input.kicad_sch (KiCad schematic)
At the start: 7 parts, among them J1 AudioJack3, U2 LM358

Commit message: First Spin of PCB
Parts:
- C1: value 1u -> 10u; JL Part# (none) -> C15850
- D1: value BAS33 -> M7; footprint Diode_THT:D_DO-35_SOD27_P7.62mm_Horizontal -> Diode_SMD:D_SMA; JL Part# (none) -> C95872
- J1: now not fitted
- R3: value 30 -> 33; JL Part# (none) -> C17634
- R4: value 10k -> 470k; JL Part# (none) -> C17709
- R5: value 22k -> 1M; JL Part# (none) -> C17514
- U2: footprint Package_DIP:DIP-8_W10.16mm -> Package_SO:SOIC-8_3.9x4.9mm_P1.27mm; JL Part# (none) -> C7950
Other:
- note added: "Gain = 3.1"
- note removed: "1uF & 32k is 32 ms Time Constant"
- note removed: "Gain = 3.2"
Changed lines of the file:
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@@
 		)
 	)
-	(text "Gain = 3.2"
+	(text "Gain = 3.1"
 		(exclude_from_sim no)
 		(at 129.54 106.68 0)
@@
 			(font
 				(size 2 2)
-			)
-			(justify left bottom)
-		)
-	)
-	(text "1uF & 32k is 32 ms\nTime Constant\n\n"
-		(exclude_from_sim no)
-		(at 172.72 104.14 0)
-		(effects
-			(font
-				(size 3 3)
 			)
 			(justify left bottom)
@@
 			)
 		)
-		(property "Value" "1u"
+		(property "Value" "10u"
 			(at 168.91 93.345 0)
 			(effects
@@
 		)
 		(property "Description" ""
+			(at 165.1 91.44 0)
+			(effects
+				(font
+					(size 1.27 1.27)
+				)
+				(hide yes)
+			)
+		)
+		(property "JL Part#" "C15850"
 			(at 165.1 91.44 0)
 			(effects
@@
 			)
 		)
-		(property "Value" "30"
+		(property "Value" "33"
 			(at 111.76 90.805 0)
 			(effects
@@
 		)
 		(property "Description" ""
+			(at 109.22 88.9 0)
+			(effects
+				(font
+					(size 1.27 1.27)
+				)
+				(hide yes)
+			)
+		)
+		(property "JL Part#" "C17634"
 			(at 109.22 88.9 0)
 			(effects
@@
 			)
 		)
-		(property "Value" "22k"
+		(property "Value" "1M"
 			(at 135.89 96.52 90)
 			(effects
@@
 		(property "Description" ""
 			(at 135.89 99.06 0)
+			(effects
+				(font
+					(size 1.27 1.27)
+				)
+				(hide yes)
+			)
+		)
+		(property "JL Part#" "C17514"
+			(at 135.89 99.06 90)
 			(effects
 				(font
@@
 			)
 		)
-		(property "Value" "10k"
+		(property "Value" "470k"
 			(at 123.19 106.045 0)
 			(effects
@@
 		)
 		(property "Description" ""
+			(at 120.65 104.14 0)
+			(effects
+				(font
+					(size 1.27 1.27)
+				)
+				(hide yes)
+			)
+		)
+		(property "JL Part#" "C17709"
 			(at 120.65 104.14 0)
 			(effects
@@
 			)
 		)
-		(property "Value" "BAS33"
+		(property "Value" "M7"
 			(at 143.51 83.82 0)
 			(effects
@@
 			)
 		)
-		(property "Footprint" "Diode_THT:D_DO-35_SOD27_P7.62mm_Horizontal"
+		(property "Footprint" "Diode_SMD:D_SMA"
 			(at 143.51 81.915 0)
 			(effects
@@
 		)
 		(property "Sim.Pins" "1=K 2=A"
+			(at 143.51 86.36 0)
+			(effects
+				(font
+					(size 1.27 1.27)
+				)
+				(hide yes)
+			)
+		)
+		(property "JL Part#" "C95872"
 			(at 143.51 86.36 0)
 			(effects
@@
 		(in_bom yes)
 		(on_board yes)
-		(dnp no)
+		(dnp yes)
 		(fields_autoplaced yes)
 		(property "Reference" "J1"
@@
 			)
 		)
-		(property "Footprint" "Package_DIP:DIP-8_W10.16mm"
+		(property "Footprint" "Package_SO:SOIC-8_3.9x4.9mm_P1.27mm"
 			(at 128.27 86.36 0)
 			(effects
@@
 			(at 128.27 86.36 0)
 			(effects
+				(font
+					(size 1.27 1.27)
+				)
+				(hide yes)
+			)
+		)
+		(property "JL Part#" "C7950"
+			(at 128.27 86.36 0)
+			(effects
