File: PCB/pulldown.kicad_sch (KiCad schematic)
At the start: 3 parts, among them Q1 2N7002

Commit message: First Spin of PCB
Parts:
- Q1: footprint Package_TO_SOT_THT:TO-92 -> Package_TO_SOT_SMD:SOT-23-3
Changed lines of the file:
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@@
 			)
 		)
-		(property "Footprint" "Package_TO_SOT_THT:TO-92"
+		(property "Footprint" "Package_TO_SOT_SMD:SOT-23-3"
 			(at 133.35 100.965 0)
 			(effects
