File: PCB/PCB.kicad_sch (KiCad schematic)
At the start: 10 parts, among them J3 Conn_02x04_Odd_Even, J5 Conn_02x04_Odd_Even, U2 LM358

Commit message: 1st draft PCB
Parts:
- added J4: Conn_01x02, Connector_PinHeader_2.54mm:PinHeader_1x02_P2.54mm_Vertical, symbol Connector_Generic:Conn_01x02
- added R14: 165, Resistor_SMD:R_0805_2012Metric_Pad1.20x1.40mm_HandSolder, symbol Device:R
Connections:
- net +5V: now also A1.4 (GPIO2), A1.5 (GPIO3), A1.6 (GPIO4), A1.7 (GPIO5)
- net CT_Input/Output: now also A1.31 (GPIO26_ADC0); no longer A1.32 (GPIO27_ADC1)
- net CT_Input1/Output: now also A1.32 (GPIO27_ADC1); no longer A1.31 (GPIO26_ADC0)
- net GND: now also R14.1
- net Pull Down/in: now also A1.20 (GPIO15); no longer A1.21 (GPIO16)
- net Pull Down1/in: now also A1.19 (GPIO14); no longer A1.22 (GPIO17)
- net Pull Down2/in: now also A1.15 (GPIO11); no longer A1.24 (GPIO18)
- net Pull Down3/in: now also A1.12 (GPIO9); no longer A1.25 (GPIO19)
- net at A1.34 (GPIO28_ADC2): now also J4.1 (Pin_1), J4.2 (Pin_2), R14.2
Other:
- moved on the sheet: A1, C3, J3, J5

Commit message: First Spin of PCB
Parts:
- added J6: Conn_01x04, Connector_PinHeader_2.54mm:PinHeader_1x04_P2.54mm_Vertical, symbol Connector_Generic:Conn_01x04
- added R16, R17: ~, Resistor_SMD:R_0805_2012Metric_Pad1.20x1.40mm_HandSolder, symbol Device:R
- A1, H1, H2, H3, H4, J3, J4, J5: now not fitted
- C2, C3: JL Part# (none) -> C28323
- R14: value 165 -> 150; JL Part# C17414 -> C17471
- U2: footprint Package_DIP:DIP-8_W10.16mm -> Package_SO:SOIC-8_3.9x4.9mm_P1.27mm; JL Part# (none) -> C7950
Connections:
- net +5V: no longer A1.4 (GPIO2), A1.5 (GPIO3), A1.6 (GPIO4), A1.7 (GPIO5)
- net GND: now also J6.2 (Pin_2)
- net +3.3V: now reaches A1.36 (3V3)
- net +3.3V: now also J6.1 (Pin_1), R16.2, R17.1
- new net SCL: A1.7 (GPIO5), J6.3 (Pin_3), R16.1
- new net SDA: A1.6 (GPIO4), J6.4 (Pin_4), R17.2

Commit message: depth working, current working
Parts:
- A1, J3, J4, J5, J6: now fitted
Changed lines of the file:
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@@
 		(in_bom yes)
 		(on_board yes)
-		(dnp yes)
+		(dnp no)
 		(fields_autoplaced yes)
 		(property "Reference" "J5"
@@
 		(in_bom yes)
 		(on_board yes)
-		(dnp yes)
+		(dnp no)
 		(fields_autoplaced yes)
 		(property "Reference" "A1"
@@
 		(in_bom yes)
 		(on_board yes)
-		(dnp yes)
+		(dnp no)
 		(property "Reference" "J6"
 			(at 85.09 66.0399 0)
@@
 		(in_bom yes)
 		(on_board yes)
-		(dnp yes)
+		(dnp no)
 		(fields_autoplaced yes)
 		(property "Reference" "J4"
@@
 		(in_bom yes)
 		(on_board yes)
-		(dnp yes)
+		(dnp no)
 		(fields_autoplaced yes)
 		(property "Reference" "J3"
